File: knuckle-pad-schemes/knuckle-pad.sch (KiCad schematic (older format))
At the start: 66 parts, among them SW1 SW_Push, SW10 SW_Push, SW11 SW_Push, SW12 SW_Push, SW13 SW_Push, SW14 SW_Push, SW15 SW_Push, SW16 SW_Push, SW17 SW_Push, SW18 SW_Push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

Commit message: updated pcb shape to (preliminary) final+added pwr_flag to schematic
Parts:
- renumbered RST to RST1
Changed lines of the file:
@@
 col5
 $Comp
-L Switch:SW_Push RST
+L Switch:SW_Push RST1
 U 1 1 611F01FE
 P 7850 2950
-F 0 "RST" H 7850 3235 50  0000 C CNN
+F 0 "RST1" H 7850 3235 50  0000 C CNN
 F 1 "SW_Push" H 7850 3144 50  0000 C CNN
 F 2 "used_footprints:Switch_Reset_THT" H 7850 3150 50  0001 C CNN
@@
 	1    0    0    -1
 $EndComp
+$Comp
+L power:PWR_FLAG #FLG0101
+U 1 1 612011BF
+P 8850 2800
+F 0 "#FLG0101" H 8850 2875 50  0001 C CNN
+F 1 "PWR_FLAG" H 8850 2973 50  0000 C CNN
+F 2 "" H 8850 2800 50  0001 C CNN
+F 3 "~" H 8850 2800 50  0001 C CNN
+	1    8850 2800
+	1    0    0    -1
+$EndComp
+$Comp
+L power:PWR_FLAG #FLG0102
+U 1 1 61201D2B
+P 9350 2800
+F 0 "#FLG0102" H 9350 2875 50  0001 C CNN
+F 1 "PWR_FLAG" H 9350 2973 50  0000 C CNN
+F 2 "" H 9350 2800 50  0001 C CNN
+F 3 "~" H 9350 2800 50  0001 C CNN
+	1    9350 2800
+	1    0    0    -1
+$EndComp
+$Comp
+L power:VCC #PWR0101
+U 1 1 61202ED4
+P 8850 2800
+F 0 "#PWR0101" H 8850 2650 50  0001 C CNN
+F 1 "VCC" H 8865 2973 50  0000 C CNN
+F 2 "" H 8850 2800 50  0001 C CNN
+F 3 "" H 8850 2800 50  0001 C CNN
+	1    8850 2800
+	-1   0    0    1
+$EndComp
+$Comp
+L power:GND #PWR0102
+U 1 1 61203DED
+P 9350 2800
+F 0 "#PWR0102" H 9350 2550 50  0001 C CNN
+F 1 "GND" H 9355 2627 50  0000 C CNN
+F 2 "" H 9350 2800 50  0001 C CNN
+F 3 "" H 9350 2800 50  0001 C CNN
+	1    9350 2800
+	1    0    0    -1
+$EndComp

Commit message: push before routing
Connections:
- net row0: now also U1.6 (3/PD0); no longer U1.2 (RX1/PD2)
- net row1: now also U1.9 (6/PD7); no longer U1.5 (2/PD1)
- no-connect marks 0 -> 8
Changed lines of the file:
@@
 	6100 850  6100 1300
 Connection ~ 6100 1300
-Text GLabel 7750 1100 0    50   Input ~ 0
+Text GLabel 7750 1500 0    50   Input ~ 0
 row0
-Text GLabel 7750 1400 0    50   Input ~ 0
+Text GLabel 7750 1800 0    50   Input ~ 0
 row1
 Text GLabel 7750 1900 0    50   Input ~ 0
@@
 	1    0    0    -1
 $EndComp
+NoConn ~ 9150 1400
+NoConn ~ 7750 1100
+NoConn ~ 7750 1000
+NoConn ~ 7750 1400
+NoConn ~ 7750 1600
+NoConn ~ 7750 1700
+NoConn ~ 9150 2100
+NoConn ~ 9150 1000
 $EndSCHEMATC
