File: knuckle-pad-schemes/knuckle-pad.sch (KiCad schematic (older format))
At the start: 66 parts, among them SW1 SW_Push, SW10 SW_Push, SW11 SW_Push, SW12 SW_Push, SW13 SW_Push, SW14 SW_Push, SW15 SW_Push, SW16 SW_Push, SW17 SW_Push, SW18 SW_Push, SW19 SW_Push, SW2 SW_Push, SW20 SW_Push, SW21 SW_Push, SW22 SW_Push, SW23 SW_Push, SW24 SW_Push, SW25 SW_Push, SW26 SW_Push, SW27 SW_Push, SW28 SW_Push, SW29 SW_Push, SW3 SW_Push, SW4 SW_Push, SW5 SW_Push, SW6 SW_Push, SW7 SW_Push, SW8 SW_Push, SW9 SW_Push, U1 ProMicro

Commit message: changed switch footprint to mx-NoLed ones
Parts:
- SW1, SW10, SW11, SW12, SW13, SW14, SW15, SW16, SW17, SW18, SW19, SW20, SW21, SW22, SW23, SW24, SW25, SW26, SW27, SW28, SW29, SW5, SW6, SW7, SW8, SW9: footprint Hybrid-Switches:MX-1u -> MX_Only:MXOnly-1U-NoLED
- SW2, SW3, SW4: footprint Hybrid-Switches:MX-1.25u -> MX_Only:MXOnly-1.25U-NoLED
Changed lines of the file:
@@
 F 0 "SW1" H 2050 1585 50  0000 C CNN
 F 1 "SW_Push" H 2050 1494 50  0000 C CNN
-F 2 "Hybrid-Switches:MX-1u" H 2050 1500 50  0001 C CNN
+F 2 "MX_Only:MXOnly-1U-NoLED" H 2050 1500 50  0001 C CNN
 F 3 "~" H 2050 1500 50  0001 C CNN
 	1    2050 1300
@@
 F 0 "SW5" H 2050 4935 50  0000 C CNN
 F 1 "SW_Push" H 2050 4844 50  0000 C CNN
-F 2 "Hybrid-Switches:MX-1u" H 2050 4850 50  0001 C CNN
+F 2 "MX_Only:MXOnly-1U-NoLED" H 2050 4850 50  0001 C CNN
 F 3 "~" H 2050 4850 50  0001 C CNN
 	1    2050 4650
@@
 F 0 "SW14" H 3650 4935 50  0000 C CNN
 F 1 "SW_Push" H 3650 4844 50  0000 C CNN
-F 2 "Hybrid-Switches:MX-1u" H 3650 4850 50  0001 C CNN
+F 2 "MX_Only:MXOnly-1U-NoLED" H 3650 4850 50  0001 C CNN
 F 3 "~" H 3650 4850 50  0001 C CNN
 	1    3650 4650
@@
 F 0 "SW19" H 4450 4935 50  0000 C CNN
 F 1 "SW_Push" H 4450 4844 50  0000 C CNN
-F 2 "Hybrid-Switches:MX-1u" H 4450 4850 50  0001 C CNN
+F 2 "MX_Only:MXOnly-1U-NoLED" H 4450 4850 50  0001 C CNN
 F 3 "~" H 4450 4850 50  0001 C CNN
 	1    4450 4650
@@
 F 0 "SW24" H 5150 4935 50  0000 C CNN
 F 1 "SW_Push" H 5150 4844 50  0000 C CNN
-F 2 "Hybrid-Switches:MX-1u" H 5150 4850 50  0001 C CNN
+F 2 "MX_Only:MXOnly-1U-NoLED" H 5150 4850 50  0001 C CNN
 F 3 "~" H 5150 4850 50  0001 C CNN
 	1    5150 4650
@@
 F 0 "SW29" H 5900 4935 50  0000 C CNN
 F 1 "SW_Push" H 5900 4844 50  0000 C CNN
-F 2 "Hybrid-Switches:MX-1u" H 5900 4850 50  0001 C CNN
+F 2 "MX_Only:MXOnly-1U-NoLED" H 5900 4850 50  0001 C CNN
 F 3 "~" H 5900 4850 50  0001 C CNN
 	1    5900 4650
@@
 F 0 "SW6" H 2850 1585 50  0000 C CNN
 F 1 "SW_Push" H 2850 1494 50  0000 C CNN
-F 2 "Hybrid-Switches:MX-1u" H 2850 1500 50  0001 C CNN
+F 2 "MX_Only:MXOnly-1U-NoLED" H 2850 1500 50  0001 C CNN
 F 3 "~" H 2850 1500 50  0001 C CNN
 	1    2850 1300
@@
 F 0 "SW10" H 3650 1585 50  0000 C CNN
 F 1 "SW_Push" H 3650 1494 50  0000 C CNN
-F 2 "Hybrid-Switches:MX-1u" H 3650 1500 50  0001 C CNN
+F 2 "MX_Only:MXOnly-1U-NoLED" H 3650 1500 50  0001 C CNN
 F 3 "~" H 3650 1500 50  0001 C CNN
 	1    3650 1300
@@
 F 0 "SW15" H 4450 1585 50  0000 C CNN
 F 1 "SW_Push" H 4450 1494 50  0000 C CNN
-F 2 "Hybrid-Switches:MX-1u" H 4450 1500 50  0001 C CNN
+F 2 "MX_Only:MXOnly-1U-NoLED" H 4450 1500 50  0001 C CNN
 F 3 "~" H 4450 1500 50  0001 C CNN
 	1    4450 1300
@@
 F 0 "SW20" H 5150 1585 50  0000 C CNN
 F 1 "SW_Push" H 5150 1494 50  0000 C CNN
-F 2 "Hybrid-Switches:MX-1u" H 5150 1500 50  0001 C CNN
+F 2 "MX_Only:MXOnly-1U-NoLED" H 5150 1500 50  0001 C CNN
 F 3 "~" H 5150 1500 50  0001 C CNN
 	1    5150 1300
@@
 F 0 "SW25" H 5900 1585 50  0000 C CNN
 F 1 "SW_Push" H 5900 1494 50  0000 C CNN
-F 2 "Hybrid-Switches:MX-1u" H 5900 1500 50  0001 C CNN
+F 2 "MX_Only:MXOnly-1U-NoLED" H 5900 1500 50  0001 C CNN
 F 3 "~" H 5900 1500 50  0001 C CNN
 	1    5900 1300
@@
 F 0 "SW2" H 2050 2385 50  0000 C CNN
 F 1 "SW_Push" H 2050 2294 50  0000 C CNN
-F 2 "Hybrid-Switches:MX-1.25u" H 2050 2300 50  0001 C CNN
+F 2 "MX_Only:MXOnly-1.25U-NoLED" H 2050 2300 50  0001 C CNN
 F 3 "~" H 2050 2300 50  0001 C CNN
 	1    2050 2100
@@
 F 0 "SW7" H 2850 2385 50  0000 C CNN
 F 1 "SW_Push" H 2850 2294 50  0000 C CNN
-F 2 "Hybrid-Switches:MX-1u" H 2850 2300 50  0001 C CNN
+F 2 "MX_Only:MXOnly-1U-NoLED" H 2850 2300 50  0001 C CNN
 F 3 "~" H 2850 2300 50  0001 C CNN
 	1    2850 2100
@@
 F 0 "SW11" H 3650 2385 50  0000 C CNN
 F 1 "SW_Push" H 3650 2294 50  0000 C CNN
-F 2 "Hybrid-Switches:MX-1u" H 3650 2300 50  0001 C CNN
+F 2 "MX_Only:MXOnly-1U-NoLED" H 3650 2300 50  0001 C CNN
 F 3 "~" H 3650 2300 50  0001 C CNN
 	1    3650 2100
@@
 F 0 "SW16" H 4450 2385 50  0000 C CNN
 F 1 "SW_Push" H 4450 2294 50  0000 C CNN
-F 2 "Hybrid-Switches:MX-1u" H 4450 2300 50  0001 C CNN
+F 2 "MX_Only:MXOnly-1U-NoLED" H 4450 2300 50  0001 C CNN
 F 3 "~" H 4450 2300 50  0001 C CNN
 	1    4450 2100
@@
 F 0 "SW21" H 5150 2385 50  0000 C CNN
 F 1 "SW_Push" H 5150 2294 50  0000 C CNN
-F 2 "Hybrid-Switches:MX-1u" H 5150 2300 50  0001 C CNN
+F 2 "MX_Only:MXOnly-1U-NoLED" H 5150 2300 50  0001 C CNN
 F 3 "~" H 5150 2300 50  0001 C CNN
 	1    5150 2100
@@
 F 0 "SW26" H 5900 2385 50  0000 C CNN
 F 1 "SW_Push" H 5900 2294 50  0000 C CNN
-F 2 "Hybrid-Switches:MX-1u" H 5900 2300 50  0001 C CNN
+F 2 "MX_Only:MXOnly-1U-NoLED" H 5900 2300 50  0001 C CNN
 F 3 "~" H 5900 2300 50  0001 C CNN
 	1    5900 2100
@@
 F 0 "SW3" H 2050 3185 50  0000 C CNN
 F 1 "SW_Push" H 2050 3094 50  0000 C CNN
-F 2 "Hybrid-Switches:MX-1.25u" H 2050 3100 50  0001 C CNN
+F 2 "MX_Only:MXOnly-1.25U-NoLED" H 2050 3100 50  0001 C CNN
 F 3 "~" H 2050 3100 50  0001 C CNN
 	1    2050 2900
@@
 F 0 "SW8" H 2850 3185 50  0000 C CNN
 F 1 "SW_Push" H 2850 3094 50  0000 C CNN
-F 2 "Hybrid-Switches:MX-1u" H 2850 3100 50  0001 C CNN
+F 2 "MX_Only:MXOnly-1U-NoLED" H 2850 3100 50  0001 C CNN
 F 3 "~" H 2850 3100 50  0001 C CNN
 	1    2850 2900
@@
 F 0 "SW12" H 3650 3185 50  0000 C CNN
 F 1 "SW_Push" H 3650 3094 50  0000 C CNN
-F 2 "Hybrid-Switches:MX-1u" H 3650 3100 50  0001 C CNN
+F 2 "MX_Only:MXOnly-1U-NoLED" H 3650 3100 50  0001 C CNN
 F 3 "~" H 3650 3100 50  0001 C CNN
 	1    3650 2900
@@
 F 0 "SW17" H 4450 3185 50  0000 C CNN
 F 1 "SW_Push" H 4450 3094 50  0000 C CNN
-F 2 "Hybrid-Switches:MX-1u" H 4450 3100 50  0001 C CNN
+F 2 "MX_Only:MXOnly-1U-NoLED" H 4450 3100 50  0001 C CNN
 F 3 "~" H 4450 3100 50  0001 C CNN
 	1    4450 2900
@@
 F 0 "SW22" H 5150 3185 50  0000 C CNN
 F 1 "SW_Push" H 5150 3094 50  0000 C CNN
-F 2 "Hybrid-Switches:MX-1u" H 5150 3100 50  0001 C CNN
+F 2 "MX_Only:MXOnly-1U-NoLED" H 5150 3100 50  0001 C CNN
 F 3 "~" H 5150 3100 50  0001 C CNN
 	1    5150 2900
@@
 F 0 "SW27" H 5900 3185 50  0000 C CNN
 F 1 "SW_Push" H 5900 3094 50  0000 C CNN
-F 2 "Hybrid-Switches:MX-1u" H 5900 3100 50  0001 C CNN
+F 2 "MX_Only:MXOnly-1U-NoLED" H 5900 3100 50  0001 C CNN
 F 3 "~" H 5900 3100 50  0001 C CNN
 	1    5900 2900
@@
 F 0 "SW4" H 2050 4035 50  0000 C CNN
 F 1 "SW_Push" H 2050 3944 50  0000 C CNN
-F 2 "Hybrid-Switches:MX-1.25u" H 2050 3950 50  0001 C CNN
+F 2 "MX_Only:MXOnly-1.25U-NoLED" H 2050 3950 50  0001 C CNN
 F 3 "~" H 2050 3950 50  0001 C CNN
 	1    2050 3750
@@
 F 0 "SW9" H 2850 4035 50  0000 C CNN
 F 1 "SW_Push" H 2850 3944 50  0000 C CNN
-F 2 "Hybrid-Switches:MX-1u" H 2850 3950 50  0001 C CNN
+F 2 "MX_Only:MXOnly-1U-NoLED" H 2850 3950 50  0001 C CNN
 F 3 "~" H 2850 3950 50  0001 C CNN
 	1    2850 3750
@@
 F 0 "SW13" H 3650 4035 50  0000 C CNN
 F 1 "SW_Push" H 3650 3944 50  0000 C CNN
-F 2 "Hybrid-Switches:MX-1u" H 3650 3950 50  0001 C CNN
+F 2 "MX_Only:MXOnly-1U-NoLED" H 3650 3950 50  0001 C CNN
 F 3 "~" H 3650 3950 50  0001 C CNN
 	1    3650 3750
@@
 F 0 "SW18" H 4450 4035 50  0000 C CNN
 F 1 "SW_Push" H 4450 3944 50  0000 C CNN
-F 2 "Hybrid-Switches:MX-1u" H 4450 3950 50  0001 C CNN
+F 2 "MX_Only:MXOnly-1U-NoLED" H 4450 3950 50  0001 C CNN
 F 3 "~" H 4450 3950 50  0001 C CNN
 	1    4450 3750
@@
 F 0 "SW23" H 5150 4035 50  0000 C CNN
 F 1 "SW_Push" H 5150 3944 50  0000 C CNN
-F 2 "Hybrid-Switches:MX-1u" H 5150 3950 50  0001 C CNN
+F 2 "MX_Only:MXOnly-1U-NoLED" H 5150 3950 50  0001 C CNN
 F 3 "~" H 5150 3950 50  0001 C CNN
 	1    5150 3750
@@
 F 0 "SW28" H 5900 4035 50  0000 C CNN
 F 1 "SW_Push" H 5900 3944 50  0000 C CNN
-F 2 "Hybrid-Switches:MX-1u" H 5900 3950 50  0001 C CNN
+F 2 "MX_Only:MXOnly-1U-NoLED" H 5900 3950 50  0001 C CNN
 F 3 "~" H 5900 3950 50  0001 C CNN
 	1    5900 3750
