File: knuckle-pad-mcuCover/knuckle-pad.kicad_pcb (KiCad board)
At the start: 2 copper layers, 128 x 115.3 mm, 28 parts, among them SW1 SW_Push, SW10 SW_Push, SW11 SW_Push, SW12 SW_Push, SW13 SW_Push, SW14 SW_Push, SW15 SW_Push, SW16 SW_Push, SW17 SW_Push, SW18 SW_Push, SW19 SW_Push, SW2 SW_Push, SW20 SW_Push, SW21 SW_Push, SW22 SW_Push, SW23 SW_Push, SW24 SW_Push, SW25 SW_Push, SW26 SW_Push, SW27 SW_Push, SW3 SW_Push, SW4 SW_Push, SW5 SW_Push, SW6 SW_Push, SW7 SW_Push, SW8 SW_Push, SW9 SW_Push, U1 ProMicro

Commit message: finalized MCU cover
Parts:
- removed SW1, SW10, SW11, SW12, SW13, SW14, SW15, SW16, SW17, SW18, SW19, SW2, SW20, SW21, SW22, SW23, SW24, SW25, SW26, SW27, SW3, SW4, SW5, SW6, SW7, SW8, SW9: SW_Push, acheron_MX_PlateSlots:MX100
- removed U1: ProMicro, Keebio-Parts:ArduinoProMicro-ZigZag
Other:
- board size 128 x 115.3 mm -> 27.2 x 40.1 mm
